File: source/main.kicad_pcb (KiCad board)
At the start: 2 copper layers, 0 parts

Commit message: Add: basic design
Parts:
- added C1: 100nF 16V X7R, lcsc:C0402, F.Cu at (0.00, 0.00)
- added C10: 100nF 16V X7R, lcsc:C0402, F.Cu at (18.7, 25.5)
- added C11: 100nF 16V X7R, lcsc:C0402, F.Cu at (8.20, 29.6)
- added C12: 100nF 16V X7R, lcsc:C0402, F.Cu at (2.46, 25.5)
- added C13: 100nF 16V X7R, lcsc:C0402, F.Cu at (2.46, 21.9)
- added C14: 100nF 16V X7R, lcsc:C0402, F.Cu at (18.7, 21.9)
- added C15: 100nF 16V X7R, lcsc:C0402, F.Cu at (8.20, 19.4)
- added C16: 100nF 16V X7R, lcsc:C0402, F.Cu at (8.60, 14.3)
- added C17: 100nF 16V X7R, lcsc:C0402, F.Cu at (1.05, 43.1)
- added C18: 100nF 16V X7R, lcsc:C0402, F.Cu at (1.05, 36.9)
- added C19: 100nF 16V X7R, lcsc:C0402, F.Cu at (4.30, 43.1)
- added C2: 18pF ±5% 50V C0G, lcsc:C0402, F.Cu at (9.00, 33.5)
- added C20: 100nF 16V X7R, lcsc:C0402, F.Cu at (4.30, 36.9)
- added C21: 100nF 16V X7R, lcsc:C0402, F.Cu at (7.55, 43.1)
- added C22: 100nF 16V X7R, lcsc:C0402, F.Cu at (7.55, 36.9)
- added C23: 100nF 16V X7R, lcsc:C0402, F.Cu at (10.8, 43.1)
- added C24: 100nF 16V X7R, lcsc:C0402, F.Cu at (10.8, 36.9)
- added C25: 100nF 16V X7R, lcsc:C0402, F.Cu at (14.1, 43.1)
- added C26: 100nF 16V X7R, lcsc:C0402, F.Cu at (14.1, 36.9)
- added C27: 100nF 16V X7R, lcsc:C0402, F.Cu at (17.3, 43.1)
- added C28: 100nF 16V X7R, lcsc:C0402, F.Cu at (17.3, 36.9)
- added C3: 18pF ±5% 50V C0G, lcsc:C0402, F.Cu at (3.00, 33.5)
- added C4: 100nF 16V X7R, lcsc:C0402, F.Cu at (3.75, 14.4)
- added C5: 10µF 25V X5R, lcsc:R0402, F.Cu at (4.93, 3.55)
- added C6: 10µF 10V X7R, lcsc:C0603, F.Cu at (11.4, 3.55)
- added C7: 100nF 16V X7R, lcsc:C0402, F.Cu at (10.6, 19.4)
- added C8: 100nF 16V X7R, lcsc:C0402, F.Cu at (8.60, 32.2)
- added C9: 100nF 16V X7R, lcsc:C0402, F.Cu at (7.80, 16.8)
- added D1: 3.05V, lcsc:LED-SMD_L3.2-W1.3-RD_GREEN-MHT151UGCT, F.Cu at (16.8, 10.0)
- added D2: 3.05V, lcsc:LED-SMD_L3.2-W1.3-RD_GREEN-MHT151UGCT, F.Cu at (13.5, 10.0)
- added J1: PICO_DebugHeader, lcsc:CONN-SMD-3P-P1.00_BM03B-SRSS-TB-LF-SN, F.Cu at (12.5, 32.5)
- added J3: Header, lcsc:HDR-TH_10P-P2.54-V-F-R2-C5-S2.54, F.Cu at (10.0, 47.5)
- added J4: Header, lcsc:HDR-TH_4P-P2.54-V-F, F.Cu at (10.0, 1.27)
- added LOGO1: faebrykLogo, custom:faebryk_logo, B.Cu at (6.00, 8.00)
- added R1: 10kΩ ±1% 62.5mW, lcsc:R0402, F.Cu at (8.75, 18.5)
- added R10: 10kΩ ±1% 62.5mW, lcsc:R0402, F.Cu at (15.0, 37.1)
- added R11: 10kΩ ±1% 62.5mW, lcsc:R0402, F.Cu at (18.2, 37.1)
- added R12: 100Ω ±1% 62.5mW, lcsc:R0402, F.Cu at (0.00, 0.00)
- added R13: 10kΩ ±1% 62.5mW, lcsc:R0402, F.Cu at (0.00, 0.00)
- added R2, R3: 1kΩ ±1% 62.5mW, lcsc:R0402, F.Cu at (6.50, 9.50)
- added R4: 1kΩ ±1% 62.5mW, lcsc:R0402, F.Cu at (7.75, 31.0)
- added R5: 1kΩ ±1% 62.5mW, lcsc:R0402, F.Cu at (16.8, 14.5)
- added R6: 1kΩ ±1% 62.5mW, lcsc:R0402, F.Cu at (13.5, 14.5)
- added R7: 10kΩ ±1% 62.5mW, lcsc:R0402, F.Cu at (5.25, 37.1)
- added R8: 10kΩ ±1% 62.5mW, lcsc:R0402, F.Cu at (8.50, 37.1)
- added R9: 10kΩ ±1% 62.5mW, lcsc:R0402, F.Cu at (11.8, 37.1)
- added S1: _Switch, lcsc:KEY-SMD_4P-L4.2-W3.2-P2.20-LS4.6, F.Cu at (4.00, 9.50)
- added S2: _Switch, lcsc:KEY-SMD_4P-L4.2-W3.2-P2.20-LS4.6, F.Cu at (9.00, 9.50)
- added U1: Wuxi_I_core_Elec_AiP74LVC1T45GB236_TR, lcsc:SOT-23-6_L2.9-W1.6-P0.95-LS2.8-BL, F.Cu at (2.00, 40.0)
- added U2: Wuxi_I_core_Elec_AiP74LVC1T45GB236_TR, lcsc:SOT-23-6_L2.9-W1.6-P0.95-LS2.8-BL, F.Cu at (5.25, 40.0)
- added U3: Wuxi_I_core_Elec_AiP74LVC1T45GB236_TR, lcsc:SOT-23-6_L2.9-W1.6-P0.95-LS2.8-BL, F.Cu at (8.50, 40.0)
- added U4: Wuxi_I_core_Elec_AiP74LVC1T45GB236_TR, lcsc:SOT-23-6_L2.9-W1.6-P0.95-LS2.8-BL, F.Cu at (11.8, 40.0)
- added U5: Winbond_W25Q16JVUXIQ, lcsc:USON-8_L3.0-W2.0-P0.50-BL-EP, F.Cu at (4.50, 17.5)
- added U6: LDO 3.3V 600mA 400mV Vin max 6V Iq 80µA, lcsc:SOT-25-5_L2.9-W1.6-P0.95-LS2.8-BL, F.Cu at (8.00, 4.50)
- added U7: RP2040, lcsc:LQFN-56_L7.0-W7.0-P0.4-EP, F.Cu at (8.00, 24.5)
- added U8: Wuxi_I_core_Elec_AiP74LVC1T45GB236_TR, lcsc:SOT-23-6_L2.9-W1.6-P0.95-LS2.8-BL, F.Cu at (15.0, 40.0)
- added U9: Wuxi_I_core_Elec_AiP74LVC1T45GB236_TR, lcsc:SOT-23-6_L2.9-W1.6-P0.95-LS2.8-BL, F.Cu at (18.2, 40.0)
- added XTAL1: Crystal, lcsc:CRYSTAL-SMD_4P-L3.2-W2.5-BL, F.Cu at (6.00, 33.5)
Routing:
- net 3V3: track 0.00 -> 35.2 mm
- net VTARGET: track 0.00 -> 8.58 mm
- net C8-1-C9-1-U7-23-U7-45-U7-50: track 0.00 -> 7.14 mm
- net VBUS: track 0.00 -> 1.34 mm
- net R9-1-U4-5: track 0.00 -> 1.32 mm
- net R8-1-U3-5: track 0.00 -> 1.32 mm
- net R7-1-U2-5: track 0.00 -> 1.32 mm
- net R11-1-U9-5: track 0.00 -> 1.32 mm
- net R10-1-U8-5: track 0.00 -> 1.32 mm
- net C7-1-U7-43: track 0.00 -> 0.99 mm
- added copper zone on B.Cu, net GND
- added copper zone on F.Cu, net GND
Other:
- board outline added: 20 x 50 mm
- board text added: "######"
- board text added: "40d324f"
- board text added: "RPDAP"
- board text added: "[ ] DAP"
- board text added: "[ ] VCP"
