File: layouts/rpdap_compact_on_board/rpdap_compact_on_board.kicad_pcb (KiCad board)
At the start: 2 copper layers, 0 parts

Commit message: refactor debug-connectors, fix issues in layout and connections
Parts:
- added CN1: , XFCN_BH254VS_20P:CONN-SMD_20P-P2.54_B-3000N20P-0110, F.Cu at (10.0, 0.00)
- added MOD1: , RPDAP_Compact:RPDAP_Compact, F.Cu at (0.00, 0.00)
- added P1: , Sinhoo_SMTSO2530CTJ:SMD_BD5.6-L5.6-W5.6-D4.1, F.Cu at (0.00, -10.0)
- added P2: , Sinhoo_SMTSO2530CTJ:SMD_BD5.6-L5.6-W5.6-D4.1, F.Cu at (0.00, -20.0)

Commit message: rebuild, small fixes, update README
Parts:
- moved CN1 24.6 mm to (0.00, 22.5), turned to 180 degrees
- moved P2 22.6 mm to (-16.1, -4.10)
- moved P1 17.1 mm to (16.1, -4.10)
