File: layouts/rpdap_stick/rpdap_stick.kicad_pcb (KiCad board)
At the start: 4 copper layers, 66 x 43.2 mm, 68 parts

Commit message: fix stick layout
Parts:
- added LOGO1: , atopile_Logo_25x6mm:atopile_Logo_25x6mm, F.Cu at (17.0, -11.2)
- moved CN1 55.8 mm to (55.5, 5.60), turned to 90 degrees
- moved C33 40.9 mm to (39.4, 18.4)
- moved LED3 36.2 mm to (28.4, 17.6), turned to 90 degrees
- moved C32 29.5 mm to (33.1, 18.4), turned to 180 degrees
- moved R8 29.1 mm to (28.8, 19.9)
- moved U15 25.3 mm to (36.2, 19.4), turned to -90 degrees
- moved LED2 9.91 mm to (31.5, 5.10), turned to -90 degrees
- moved R1 2.93 mm to (31.5, 2.52), turned to 90 degrees
Connections:
- net vcp_indicator-power-GND-0 renamed GND
- USB1 pad : connector-net -> (no net)
Routing:
- net GND: track 0.00 -> 142.8 mm, vias 0 -> 36
- net (no net): track 127.2 -> 0.00 mm, vias 39 -> 22
- net vcp_indicator-power-GND-1: track 121.3 -> 0.00 mm, vias 33 -> 0
- net SCL: track 48.1 -> 0.00 mm, vias 2 -> 0
- net TDI: track 0.00 -> 28.0 mm, vias 0 -> 2
- net a-TX: track 0.00 -> 23.2 mm, vias 0 -> 2
- net uart-RX: track 0.00 -> 18.3 mm, vias 0 -> 2
- net model-a-line-4: track 0.00 -> 16.0 mm, vias 0 -> 1
- net a-RX: track 0.00 -> 13.4 mm, vias 0 -> 2
- net reference-VCC: track 51.1 -> 64.5 mm, vias 0 -> 2
- net TMS_DIO: track 0.00 -> 12.1 mm, vias 0 -> 2
- net TCK_SWCLK: track 0.00 -> 10.2 mm, vias 0 -> 2
- net TDO_SWO: track 0.00 -> 9.32 mm, vias 0 -> 2
- net uart-TX: track 0.00 -> 9.08 mm, vias 0 -> 2
- net nRESET: track 0.00 -> 9.04 mm, vias 0 -> 2
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- added copper zone on In2.Cu, net (none)
- added copper zone on B.Cu, net GND
- added copper zone on F.Cu, net GND
- added copper zone on In2.Cu, net GND
- removed copper zone on B.Cu, net vcp_indicator-power-GND-1
- removed copper zone on F.Cu, net vcp_indicator-power-GND-1
- removed copper zone on In2.Cu, net vcp_indicator-power-GND-1
Other:
- board text added: "RST TDI TDO/SWO TCK/CLK TMS/DIO"
- board text removed: "RST - SWO CLK DIO"
- board text removed: "VCP PWR"

Commit message: rebuild, small fixes, update README
Connections:
- U3 pad 5: (no net) -> 3V3
- U5 pad 5: (no net) -> 3V3
- U6 pad 5: (no net) -> 3V3
- U7 pad 5: (no net) -> 3V3
- USB1 pad : (no net) -> connector-net
Other:
- board text added: "{{GITHASH}}"

Commit message: fix: Update deps, swapped pinout (#2)
* rebuild with upstream rp2040 fixes. move header .25mm to the right. center dap-LED

* fix workflow triggers

* fix swapped jlink connector pinout + update deps

* pin atopile workflow version to v1.x.x
Parts:
- removed C32, C33: 100nF ±10% 16V X7R, Samsung_Electro_Mechanics_CL05B104KO5NNNC:C0402
- removed R13, R14: 5.1kΩ ±1% 62.5mW, UNI_ROYAL_0402WGF5101TCE:R0402
- added R10: 5.1kΩ ±1% 62.5mW, UNI_ROYAL_0402WGF5101TCE:R0402, F.Cu at (9.75, 14.6)
- added R9: 5.1kΩ ±1% 62.5mW, UNI_ROYAL_0402WGF5101TCE:R0402, F.Cu at (9.75, 8.85)
- C15, C30: value 1µF ±10% 25V X5R -> 100nF ±10% 16V X7R; footprint Samsung_Electro_Mechanics_CL05A105KA5NQNC:C0402 -> Samsung_Electro_Mechanics_CL05B104KO5NNNC:C0402
- C16, C28: value 2.2µF ±20% 6.3V X5R -> 100nF ±10% 16V X7R; footprint Samsung_Electro_Mechanics_CL05A225MQ5NSNC:C0402 -> Samsung_Electro_Mechanics_CL05B104KO5NNNC:C0402
- C17, C22, C29: value 100nF ±10% 16V X7R -> 2.2µF ±10% 16V X5R; footprint Samsung_Electro_Mechanics_CL05B104KO5NNNC:C0402 -> Samsung_Electro_Mechanics_CL05A225KO5NQNC:C0402
- C19: value 15pF ±5% 50V C0G -> 100nF ±10% 16V X7R; footprint FH_0402CG150J500NT:C0402 -> Samsung_Electro_Mechanics_CL05B104KO5NNNC:C0402
- C21: value 2.2µF ±20% 6.3V X5R -> 15pF ±5% 50V C0G; footprint Samsung_Electro_Mechanics_CL05A225MQ5NSNC:C0402 -> FH_0402CG150J500NT:C0402
- R1, R3: value 1kΩ ±1% 62.5mW -> 10kΩ ±1% 62.5mW; footprint UNI_ROYAL_0402WGF1001TCE:R0402 -> UNI_ROYAL_0402WGF1002TCE:R0402
- R2: value 10kΩ ±1% 62.5mW -> 1kΩ ±1% 62.5mW; footprint UNI_ROYAL_0402WGF1002TCE:R0402 -> UNI_ROYAL_0402WGF1001TCE:R0402
- R5: value 10kΩ ±1% 62.5mW -> 27Ω ±1% 62.5mW; footprint UNI_ROYAL_0402WGF1002TCE:R0402 -> UNI_ROYAL_0402WGF270JTCE:R0402
- R6: footprint YAGEO_RC0402FR_0727RL:R0402 -> UNI_ROYAL_0402WGF270JTCE:R0402
- R7: value 27Ω ±1% 62.5mW -> 1kΩ ±1% 62.5mW; footprint YAGEO_RC0402FR_0727RL:R0402 -> UNI_ROYAL_0402WGF1001TCE:R0402
- X1: footprint Yangxing_Tech_X322512MSB4SI:CRYSTAL-SMD_4P-L3.2-W2.5-BL -> Abracon_LLC_ABM8_272_T3:CRYSTAL-SMD_4P-L3.2-W2.5-BL
- moved C30 24.4 mm to (18.2, 18.6), turned to -90 degrees
- moved R2 21.6 mm to (36.9, 9.45), turned to 180 degrees
- moved C16 19.0 mm to (39.4, 18.4), turned to 0 degrees
- moved C21 16.4 mm to (39.1, 9.45), turned to 0 degrees
- moved R5 16.1 mm to (24.8, 5.10)
- moved R1 16.0 mm to (25.2, 17.2)
- moved C28 15.1 mm to (30.0, 17.4)
- moved C15 14.9 mm to (33.1, 18.4), turned to 180 degrees
- moved C23 12.3 mm to (22.5, 10.1), turned to 180 degrees
- moved R4 12.2 mm to (39.8, 7.10), turned to 90 degrees
- moved C26 12.1 mm to (30.0, 5.85), turned to 90 degrees
- moved C18 12.0 mm to (22.8, 11.1), turned to 180 degrees
- moved R3 10.9 mm to (28.4, 2.60), turned to -90 degrees
- moved C24 10.1 mm to (34.8, 11.2), turned to 0 degrees
- moved R7 6.30 mm to (31.5, 2.52), turned to 90 degrees
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Connections:
- net A renamed input-A
- net _power_vbus-VCC renamed Vbus_fused
- net a-RX renamed mcu-uart-RX
- net a-TX renamed mcu-uart-TX
- net dir-line renamed DIR
- net model-a-line-0 renamed gpio[12]-A
- net model-a-line-1 renamed gpio[11]-A
- net model-a-line-2 renamed gpio[14]-A
- net model-a-line-3 renamed gpio[15]-A
- net model-a-line-4 renamed gpio[13]-A
- net uart-RX renamed uart_connector-uart-RX
- net uart-TX renamed uart_connector-uart-TX
- C15 pad 1: chip_select -> 3V3
- C16 pad 1: _core_regulator_out_power-VCC -> reference-VCC
- C19 pad 1: XIN -> _core_regulator_out_power-VCC
- C20 pad 1: output -> XIN
- C21 pad 1: 3V3 -> output
- C30 pad 1: RUN -> 3V3
- D1 pad 1: USB_N -> input-USB_D_N
- D1 pad 3: USB_P -> input-USB_D_P
- D1 pad 4: USB_P -> input-USB_D_P
- D1 pad 6: USB_N -> input-USB_D_N
- R1 pad 1: footprint-cathode-0 -> chip_select
- R1 pad 2: GND -> 3V3
- R2 pad 1: 3V3 -> output
- R2 pad 2: chip_select -> XOUT
- R3 pad 1: output -> GND
- R3 pad 2: XOUT -> K
- R4 pad 1: GND -> RUN
- R4 pad 2: K -> 3V3
- R5 pad 1: 3V3 -> input-USB_D_P
- R5 pad 2: RUN -> output-USB_D_P
- R6 pad 1: USB_P -> input-USB_D_N
- R6 pad 2: RP_USB_P -> output-USB_D_N
- R7 pad 1: USB_N -> footprint-cathode-0
- R7 pad 2: RP_USB_N -> GND
- SW1 pad 1: GND -> chip_select
- SW1 pad 2: GND -> chip_select
- SW1 pad 3: chip_select -> GND
- SW1 pad 4: chip_select -> GND
- SW2 pad 1: GND -> RUN
- SW2 pad 2: GND -> RUN
- SW2 pad 3: RUN -> GND
- SW2 pad 4: RUN -> GND
- U8 pad 46: RP_USB_N -> output-USB_D_N
- U8 pad 47: RP_USB_P -> output-USB_D_P
- USB1 pad 5: USB_N -> input-USB_D_N
- USB1 pad 6: USB_P -> input-USB_D_P
- USB1 pad 7: USB_N -> input-USB_D_N
- USB1 pad 8: USB_P -> input-USB_D_P
Routing:
- net input-USB_D_N: track 0.00 -> 28.0 mm, vias 0 -> 2
- net USB_N: track 28.0 -> 0.00 mm, vias 2 -> 0
- net USB_P: track 26.4 -> 0.00 mm, vias 2 -> 0
- net input-USB_D_P: track 0.00 -> 26.4 mm, vias 0 -> 2
- net output-USB_D_P: track 0.00 -> 7.78 mm, vias 0 -> 2
- net RP_USB_P: track 7.78 -> 0.00 mm, vias 2 -> 0
- net RP_USB_N: track 7.11 -> 0.00 mm, vias 2 -> 0
- net output-USB_D_N: track 0.00 -> 7.11 mm, vias 0 -> 2
- net GND: track 142.8 -> 140.6 mm, vias 36 -> 38
- net chip_select: track 12.9 -> 10.8 mm
- net uart_connector-uart-RX: track 18.3 -> 19.4 mm, vias 2 -> 3
- net TDI: track 28.0 -> 29.2 mm, vias 2 -> 3
- net RUN: track 9.61 -> 8.61 mm
- net 3V3: track 64.7 -> 63.9 mm
- net (no net): vias 22 -> 21
- added copper zone on In1.Cu, net (none)
Other:
- outline, holes or cut-outs redrawn
- board text added: "V0.1.2"
- board text removed: "V0.1.0"
